File: 60.kicad_pcb (KiCad board)
At the start: 2 copper layers, 121 parts, among them SW0:0 TILDE, SW0:1 1, SW0:10 10, SW0:11 -, SW0:12 =, SW0:13 BACKSPACE, SW0:2 2, SW0:3 3, SW0:4 4, SW0:5 5, SW0:6 6, SW0:7 7, SW0:8 8, SW0:9 9, SW1:0 TAB, SW1:1 Q, SW1:10 P, SW1:11 [, SW1:12 ], SW1:13 \, SW1:2 W, SW1:3 E, SW1:4 R, SW1:5 T, SW1:6 Y, SW1:7 U, SW1:8 I, SW1:9 O, SW2:0 CAP, SW2:1 A, SW2:10 ;, SW2:11 ', SW2:12 ENTER, SW2:2 S, SW2:3 D, SW2:4 F, SW2:5 G, SW2:6 H, SW2:7 J, SW2:8 K, SW2:9 L, SW3:0 SHIFT, SW3:1 Z, SW3:10 /, SW3:11 RIGHT SHIFT, SW3:2 X, SW3:3 C, SW3:4 V, SW3:5 B, SW3:6 N, SW3:7 M, SW3:8 ,, SW3:9 ., SW4:0 LEFT_CTRL, SW4:1 FN, SW4:10 RIGHT_CONTROL, SW4:2 LEFT_ALT, SW4:7 SPACE, SW4:8 RIGHT_ALT, SW4:9 RIGHT_FN, U1 TEENSY2.0

Commit message: Updated for a smaller PCB footprint
Parts:
- moved D55 21.8 mm to (263.4, 125.9), turned to 270 degrees
- moved D20 15.2 mm to (144.8, 135.2)
- moved D57 1.83 mm to (273.9, 78.1)
- moved D10 1.65 mm to (65.1, 135.4)
- moved D5 1.53 mm to (41.3, 135.3)
- moved D21 0.76 mm to (114.3, 58.9)
- moved D41 0.76 mm to (232.4, 135.1)
- moved D51 0.71 mm to (280.7, 135.2)
- moved D11 0.66 mm to (76.2, 59.0)
- moved D53 0.62 mm to (256.4, 78.1)
- moved D60 0.61 mm to (294.2, 78.3)
- moved D46 0.61 mm to (256.5, 135.3)
- moved D6 0.61 mm to (57.1, 59.1)
- moved D25 0.56 mm to (133.3, 59.1)
- moved D29 0.56 mm to (152.4, 59.1)
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Routing:
- net /COL11: track 202.2 -> 228.8 mm
- net /COL5: track 108.9 -> 124.1 mm
- net Net-(D20-Pad1): track 5.08 -> 17.6 mm
- net Net-(D55-Pad1): track 5.08 -> 15.1 mm
- net /COL0: track 251.7 -> 246.8 mm
- net /COL2: track 185.0 -> 180.3 mm
- net /COL1: track 225.6 -> 222.9 mm
- net /COL12: track 189.9 -> 192.1 mm
- net Net-(D57-Pad1): track 5.08 -> 6.41 mm
- net Net-(D10-Pad1): track 5.08 -> 6.24 mm
- net Net-(D5-Pad1): track 5.08 -> 6.23 mm
Other:
- board outline added: 284.2 x 99.4 mm
